File: pcb_medusa/pcb_medusa.kicad_sch (KiCad schematic)
At the start: 1 part

Commit message: update
Parts:
- added C1, C3: 10uF, symbol Device:C_Polarized
- added C2, C4: 0.1uF, symbol Device:C
- added D1, D2, D3: 1N5819, Diode_THT:D_DO-41_SOD81_P10.16mm_Horizontal, symbol Diode:1N5819
- added J1: Conn_01x03_Pin, symbol Connector:Conn_01x03_Pin
- added R1: R, symbol Device:R
- added SW1: SW_SPST, symbol Switch:SW_SPST
- added U1: 74AHCT125, symbol 74xx:74AHCT125
- ESP32_S1: footprint (none) -> Espressif:ESP32-S3-ZERO
Connections:
- new net: D2.1 (K), J1.2 (Pin_2)
- new net: C3.1, C4.2, D3.1 (K), J1.3 (Pin_3)
- new net: D1.1 (K), SW1.1 (A)
- new net: C1.1, C2.1, ESP32_S1.1 (5V), SW1.2 (B)
- new net: R1.2, U1.2
- new net: D2.2 (A), U1.3
- new net: ESP32_S1.10 (7), R1.1
- new net +5V: D1.2 (A), D3.2 (A), U1.14 (VCC)
- new net GND: C1.2, C2.2, C3.2, C4.1, ESP32_S1.2 (GND), J1.1 (Pin_1), U1.1, U1.7 (GND)
- no-connect marks 0 -> 9
